File: stm32pcb.kicad_pcb (KiCad board)
At the start: 2 copper layers, 11 parts, among them J1 USB_C_Receptacle_USB2.0_16P, J2 Conn_01x04_Pin, J3 USB_C_Receptacle_USB2.0_16P, SW2 SW_Push_DPDT, U1 STM32F103C_8-B_Tx, U2 CH340C, U3 AMS1117-3.3

Commit message: 2
Parts:
- moved U3 4.20 mm to (149.7, 58.9)
Changed lines of the file:
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@@
 	(footprint "Package_TO_SOT_SMD:SOT-223-3_TabPin2"
 		(layer "F.Cu")
-		(at 153.85 59.56)
+		(at 149.7 58.9375)
 		(descr "module CMS SOT223 4 pins")
 		(tags "CMS SOT")

Commit message: update
Parts:
- added C3: 100nF, Capacitor_SMD:C_0805_2012Metric, F.Cu at (191.2, 86.7)
- added C4: 22p, Capacitor_SMD:C_0805_2012Metric, F.Cu at (191.2, 89.7)
- added C5: 22p, Capacitor_SMD:C_0805_2012Metric, F.Cu at (191.2, 92.7)
- added C6: 12pF, Capacitor_SMD:C_0805_2012Metric, F.Cu at (191.2, 95.7)
- added C7: 12pF, Capacitor_SMD:C_0805_2012Metric, F.Cu at (191.2, 98.7)
- added SW1: SW_Push_DPDT, lcsc:SW-SMD_6P-L9.1-W3.5-P2.50, F.Cu at (202.2, 83.6)
- added Y1: 8MHz, Crystal:Crystal_SMD_3225-4Pin_3.2x2.5mm, F.Cu at (196.1, 93.0)
- added Y2: 32.768kHz, Crystal:Crystal_SMD_3215-2Pin_3.2x1.5mm, F.Cu at (196.0, 97.0)
- C1: value 10u -> 10uF
- C2: value 22u -> 22uF
- R1, R2: value R -> 5.1kΩ
Connections:
- J2 pad 2: unconnected-(J2-Pin_2-Pad2) -> GND
- J2 pad 3: unconnected-(J2-Pin_3-Pad3) -> SWDIO
- J2 pad 4: unconnected-(J2-Pin_4-Pad4) -> SWCLK

Commit message: update
Parts:
- added C10: 100nF, Capacitor_SMD:C_0805_2012Metric, F.Cu at (113.5, 117.8)
- added C11: 100nF, Capacitor_SMD:C_0805_2012Metric, F.Cu at (113.5, 120.8)
- added C12: 100nF, Capacitor_SMD:C_0805_2012Metric, F.Cu at (113.5, 123.8)
- added C8: 100nF, Capacitor_SMD:C_0805_2012Metric, F.Cu at (113.5, 111.8)
- added C9: 100nF, Capacitor_SMD:C_0805_2012Metric, F.Cu at (113.5, 114.8)
- added D1: LED, LED_SMD:LED_0805_2012Metric, F.Cu at (118.0, 116.0)
- added D2: LED, LED_SMD:LED_0805_2012Metric, F.Cu at (118.0, 119.0)
- added J4: Conn_01x12_Pin, Connector_PinHeader_2.54mm:PinHeader_1x12_P2.54mm_Vertical, F.Cu at (87.1, 116.5)
- added R3: 10kΩ, Resistor_SMD:R_1206_3216Metric, F.Cu at (108.5, 111.9)
- added R4: 10kΩ, Resistor_SMD:R_1206_3216Metric, F.Cu at (108.5, 115.2)
- added R5: 1kΩ, Resistor_SMD:R_1206_3216Metric, F.Cu at (108.5, 118.5)
- added R6: 1kΩ, Resistor_SMD:R_1206_3216Metric, F.Cu at (108.5, 121.8)
- added R7: 10kΩ, Resistor_SMD:R_1206_3216Metric, F.Cu at (108.5, 125.1)
- added R8: 1.5kΩ, Resistor_SMD:R_1206_3216Metric, F.Cu at (108.5, 128.5)
- added SW3: SW_Push_DPDT, Button_Switch_SMD:SW_DPDT_CK_JS202011JCQN, F.Cu at (116.5, 128.1)
- added SW4: SW_Push_DPDT, Button_Switch_SMD:SW_DPDT_CK_JS202011JCQN, F.Cu at (116.5, 133.6)
- added SW5: TS-1088-AR02016, lcsc:SW-SMD_L3.9-W3.0-P4.45, F.Cu at (119.0, 112.4)
Connections:
- J1 pad A6: unconnected-(J1-D+-PadA6) -> USB_DP
- J1 pad A7: unconnected-(J1-D--PadA7) -> USB_DN
- J1 pad B6: unconnected-(J1-D+-PadB6) -> USB_DP
- J1 pad B7: unconnected-(J1-D--PadB7) -> USB_DN
- U1 pad 20: unconnected-(U1-PB2-Pad20) -> PB2_BOOT1
- U1 pad 23: Net-(U1-VSS-Pad23) -> GND
- U1 pad 24: unconnected-(U1-VDD-Pad24) -> STM32_3V3
- U1 pad 35: Net-(U1-VSS-Pad23) -> GND
- U1 pad 36: unconnected-(U1-VDD-Pad36) -> STM32_3V3
- U1 pad 44: unconnected-(U1-BOOT0-Pad44) -> BOOT0
- U1 pad 47: Net-(U1-VSS-Pad23) -> GND
- U1 pad 48: unconnected-(U1-VDD-Pad48) -> STM32_3V3
- U1 pad 7: unconnected-(U1-NRST-Pad7) -> NRST
- U1 pad 8: unconnected-(U1-VSSA-Pad8) -> GND
- U1 pad 9: unconnected-(U1-VDDA-Pad9) -> STM32_3V3

Commit message: update
Parts:
- added C13: 100nF, Capacitor_SMD:C_0805_2012Metric, B.Cu at (151.0, 83.3)
- added C14: 100nF, Capacitor_SMD:C_0805_2012Metric, B.Cu at (154.3, 81.1)
- added J5: Conn_01x12_Pin, Connector_PinHeader_2.54mm:PinHeader_1x12_P2.54mm_Vertical, F.Cu at (208.4, 67.8)
- added J6: Conn_01x12_Pin, Connector_PinHeader_2.54mm:PinHeader_1x12_P2.54mm_Vertical, F.Cu at (176.8, 71.5)
- added J7: Conn_01x12_Pin, Connector_PinHeader_2.54mm:PinHeader_1x12_P2.54mm_Vertical, F.Cu at (180.5, 103.2)
- added R10: 5.1kΩ, Resistor_SMD:R_1206_3216Metric, B.Cu at (144.9, 87.0)
- added R11: 220Ω, Resistor_SMD:R_1206_3216Metric, B.Cu at (155.6, 83.7)
- added R12: 220Ω, Resistor_SMD:R_1206_3216Metric, B.Cu at (155.6, 86.3)
- added R9: 5.1kΩ, Resistor_SMD:R_1206_3216Metric, B.Cu at (144.9, 84.0)
- C10, C11, C12, C3, C8, C9, R1, R2, R7: moved to B.Cu
- SW2, SW3, SW4: footprint Button_Switch_SMD:SW_DPDT_CK_JS202011JCQN -> lcsc:SW-SMD_6P-L9.1-W3.5-P2.50
- moved J4 126.2 mm to (212.2, 99.5), turned to 180 degrees
- moved C10 90.7 mm to (198.2, 85.2), turned to 90 degrees
- moved C11 87.4 mm to (191.5, 81.5)
- moved D1 87.3 mm to (92.4, 32.6)
- moved C9 86.7 mm to (196.5, 89.7), turned to 180 degrees
- moved R5 85.9 mm to (98.2, 33.2)
- moved U1 83.1 mm to (194.0, 85.7), turned to 180 degrees
- moved D2 81.0 mm to (92.4, 42.2)
- moved R6 81.0 mm to (99.1, 41.4)
- moved C8 79.9 mm to (189.8, 88.1), turned to 90 degrees
- moved R7 78.9 mm to (167.6, 72.9), turned to 180 degrees
- moved C12 76.1 mm to (167.5, 70.1), turned to 180 degrees
- moved R8 74.6 mm to (153.3, 68.8)
- moved SW5 64.2 mm to (167.6, 70.5)
- moved J1 52.2 mm to (144.7, 72.0), turned to -90 degrees
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Connections:
- J3 pad A1: Net-(J3-GND-PadA1) -> GND
- J3 pad A12: Net-(J3-GND-PadA1) -> GND
- J3 pad A4: Net-(J3-VBUS-PadA4) -> CH340_USB_VBUS
- J3 pad A5: unconnected-(J3-CC1-PadA5) -> Net-(J3-CC1)
- J3 pad A6: unconnected-(J3-D+-PadA6) -> CH340_USB_DP
- J3 pad A7: unconnected-(J3-D--PadA7) -> CH340_USB_DN
- J3 pad A9: Net-(J3-VBUS-PadA4) -> CH340_USB_VBUS
- J3 pad B1: Net-(J3-GND-PadA1) -> GND
- J3 pad B12: Net-(J3-GND-PadA1) -> GND
- J3 pad B4: Net-(J3-VBUS-PadA4) -> CH340_USB_VBUS
- J3 pad B5: unconnected-(J3-CC2-PadB5) -> Net-(J3-CC2)
- J3 pad B6: unconnected-(J3-D+-PadB6) -> CH340_USB_DP
- J3 pad B7: unconnected-(J3-D--PadB7) -> CH340_USB_DN
- J3 pad B9: Net-(J3-VBUS-PadA4) -> CH340_USB_VBUS
- J3 pad S1: unconnected-(J3-SHIELD-PadS1) -> GND
- J4 pad 1: unconnected-(J4-Pin_1-Pad1) -> Net-(J4-Pin_1)
- J4 pad 10: unconnected-(J4-Pin_10-Pad10) -> Net-(J4-Pin_10)
- J4 pad 11: unconnected-(J4-Pin_11-Pad11) -> Net-(J4-Pin_11)
- J4 pad 12: unconnected-(J4-Pin_12-Pad12) -> Net-(J4-Pin_12)
- J4 pad 2: unconnected-(J4-Pin_2-Pad2) -> Net-(J4-Pin_2)
- J4 pad 4: unconnected-(J4-Pin_4-Pad4) -> OSC32_OUT
- J4 pad 5: unconnected-(J4-Pin_5-Pad5) -> OSC_IN
- J4 pad 6: unconnected-(J4-Pin_6-Pad6) -> OSC_OUT
- J4 pad 7: unconnected-(J4-Pin_7-Pad7) -> NRST
- J4 pad 8: unconnected-(J4-Pin_8-Pad8) -> GND
- J4 pad 9: unconnected-(J4-Pin_9-Pad9) -> STM32_3V3
- U1 pad 1: unconnected-(U1-VBAT-Pad1) -> Net-(J4-Pin_1)
- U1 pad 10: unconnected-(U1-PA0-Pad10) -> Net-(J4-Pin_10)
- U1 pad 11: unconnected-(U1-PA1-Pad11) -> Net-(J4-Pin_11)
- U1 pad 12: unconnected-(U1-PA2-Pad12) -> Net-(J4-Pin_12)
- U1 pad 13: unconnected-(U1-PA3-Pad13) -> Net-(J5-Pin_1)
- U1 pad 14: unconnected-(U1-PA4-Pad14) -> Net-(J5-Pin_2)
- U1 pad 15: unconnected-(U1-PA5-Pad15) -> Net-(J5-Pin_3)
- U1 pad 16: unconnected-(U1-PA6-Pad16) -> Net-(J5-Pin_4)
- U1 pad 17: unconnected-(U1-PA7-Pad17) -> Net-(J5-Pin_5)
- U1 pad 18: unconnected-(U1-PB0-Pad18) -> Net-(J5-Pin_6)
- U1 pad 19: unconnected-(U1-PB1-Pad19) -> Net-(J5-Pin_7)
- U1 pad 2: unconnected-(U1-PC13-Pad2) -> Net-(J4-Pin_2)
- U1 pad 21: unconnected-(U1-PB10-Pad21) -> Net-(J5-Pin_9)
- U1 pad 22: unconnected-(U1-PB11-Pad22) -> Net-(J5-Pin_10)
- U1 pad 25: unconnected-(U1-PB12-Pad25) -> Net-(J6-Pin_1)
- U1 pad 26: unconnected-(U1-PB13-Pad26) -> Net-(J6-Pin_2)
- U1 pad 27: unconnected-(U1-PB14-Pad27) -> Net-(J6-Pin_3)
- U1 pad 28: unconnected-(U1-PB15-Pad28) -> Net-(J6-Pin_4)
- U1 pad 29: unconnected-(U1-PA8-Pad29) -> Net-(J6-Pin_5)
- U1 pad 3: unconnected-(U1-PC14-Pad3) -> OSC32_IN
- U1 pad 30: unconnected-(U1-PA9-Pad30) -> CH340_RX
- U1 pad 31: unconnected-(U1-PA10-Pad31) -> CH340_TX
- U1 pad 32: unconnected-(U1-PA11-Pad32) -> USB_DN
- U1 pad 33: unconnected-(U1-PA12-Pad33) -> USB_DP
- U1 pad 34: unconnected-(U1-PA13-Pad34) -> SWDIO
- U1 pad 37: unconnected-(U1-PA14-Pad37) -> SWCLK
- U1 pad 38: unconnected-(U1-PA15-Pad38) -> Net-(J7-Pin_2)
- U1 pad 39: unconnected-(U1-PB3-Pad39) -> Net-(J7-Pin_3)
- U1 pad 4: unconnected-(U1-PC15-Pad4) -> OSC32_OUT
- U1 pad 40: unconnected-(U1-PB4-Pad40) -> Net-(J7-Pin_4)
- U1 pad 41: unconnected-(U1-PB5-Pad41) -> Net-(J7-Pin_5)
- U1 pad 42: unconnected-(U1-PB6-Pad42) -> Net-(J7-Pin_6)
- U1 pad 43: unconnected-(U1-PB7-Pad43) -> Net-(J7-Pin_7)
- U1 pad 45: unconnected-(U1-PB8-Pad45) -> Net-(J7-Pin_9)
- U1 pad 46: unconnected-(U1-PB9-Pad46) -> Net-(J7-Pin_10)
- U1 pad 5: unconnected-(U1-PD0-Pad5) -> OSC_IN
- U1 pad 6: unconnected-(U1-PD1-Pad6) -> OSC_OUT
- U2 pad 1: unconnected-(U2-GND-Pad1) -> GND
- U2 pad 16: unconnected-(U2-VCC-Pad16) -> CH340_USB_VBUS
- U2 pad 2: unconnected-(U2-TXD-Pad2) -> Net-(U2-TXD)
- U2 pad 3: unconnected-(U2-RXD-Pad3) -> Net-(U2-RXD)
- U2 pad 4: unconnected-(U2-V3-Pad4) -> Net-(U2-V3)
- U2 pad 5: unconnected-(U2-UD+-Pad5) -> CH340_USB_DP
- U2 pad 6: unconnected-(U2-UD--Pad6) -> CH340_USB_DN

Commit message: update
Parts:
- C1, C2, R3, R4, R5, R6, R8, SW3, SW4, U3: moved to B.Cu
- moved R3 87.9 mm to (183.8, 96.8), turned to 180 degrees
- moved SW3 86.4 mm to (190.9, 96.8), turned to 180 degrees
- moved R4 85.8 mm to (192.5, 96.8), turned to 180 degrees
- moved SW4 82.7 mm to (182.2, 96.8), turned to 180 degrees
- moved D2 81.8 mm to (170.1, 67.7)
- moved D1 77.5 mm to (161.4, 67.8)
- moved R6 76.2 mm to (170.7, 67.6), turned to 180 degrees
- moved R5 72.6 mm to (162.1, 67.7), turned to 180 degrees
- moved C2 72.6 mm to (193.2, 76.2), turned to -90 degrees
- moved U3 70.1 mm to (187.4, 74.6)
- moved SW2 60.7 mm to (170.4, 74.1)
- moved C1 58.5 mm to (181.5, 74.5), turned to -90 degrees
- moved R7 31.9 mm to (199.5, 72.4), turned to 0 degrees
- moved C12 28.5 mm to (195.7, 74.4), turned to -90 degrees
- moved SW5 21.6 mm to (188.9, 74.5), turned to 90 degrees
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Routing:
- net GND: track 0.00 -> 46.1 mm, vias 0 -> 33
- net OSC32_OUT: track 0.00 -> 8.88 mm
- net OSC32_IN: track 0.00 -> 8.80 mm
- net OSC_IN: track 0.00 -> 7.54 mm
- net OSC_OUT: track 0.00 -> 7.44 mm

Commit message: update
Parts:
- J1, J3: footprint Connector_USB:USB_C_Receptacle_GCT_USB4105-xx-A_16P_TopMnt_Horizontal -> lcsc:USB-C-SMD_HH-16P-CB-TYPE-C
- SW5: moved to B.Cu
- moved C2 28.8 mm to (169.4, 92.6), turned to 180 degrees
- moved U3 20.4 mm to (171.0, 86.8), turned to -90 degrees
- moved R1 18.6 mm to (162.9, 91.3), turned to -90 degrees
- moved R9 15.4 mm to (163.7, 68.7), turned to 90 degrees
- moved SW2 13.6 mm to (165.9, 86.9), turned to 180 degrees
- moved R6 13.5 mm to (165.5, 80.2), turned to -90 degrees
- moved R8 13.5 mm to (165.9, 86.3)
- moved R12 13.4 mm to (171.6, 72.6)
- moved C14 13.4 mm to (170.3, 67.4)
- moved R11 13.4 mm to (171.6, 70.0)
- moved C13 13.4 mm to (167.0, 69.6)
- moved U2 13.4 mm to (170.2, 72.3)
- moved D2 13.2 mm to (165.5, 80.1), turned to -90 degrees
- moved J1 13.2 mm to (158.4, 87.2)
- moved R10 13.1 mm to (163.7, 74.1), turned to -90 degrees
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Connections:
- R4 pad 1: BOOT0 -> PB2_BOOT1
Routing:
- net GND: track 46.1 -> 86.3 mm, vias 33 -> 36
- net USB_DN: track 0.00 -> 36.4 mm, vias 0 -> 3
- net USB_DP: track 0.00 -> 36.3 mm, vias 0 -> 3
- net Net-(U3-VI): track 0.00 -> 17.3 mm, vias 0 -> 1
- net USB_VBUS: track 0.00 -> 14.0 mm
- net REG_3V3: track 0.00 -> 9.20 mm, vias 0 -> 2
- net Net-(J1-CC1): track 0.00 -> 3.02 mm, vias 0 -> 1
- net Net-(J1-CC2): track 0.00 -> 2.56 mm, vias 0 -> 1
- net CH340_USB_DP: track 0.00 -> 0.13 mm, vias 0 -> 1
- net CH340_USB_DN: vias 0 -> 1
Other:
- board outline added: 61.1 x 40.7 mm

Commit message: update
Parts:
- moved R10 1.27 mm to (164.6, 75.0)
- moved R9 0.83 mm to (163.6, 69.5)
- moved D1 0.13 mm to (162.6, 80.2)
- moved R5 0.13 mm to (162.6, 80.3)
- moved J3 0.13 mm to (158.4, 73.5)
Routing:
- net CH340_USB_VBUS: track 0.00 -> 37.3 mm, vias 0 -> 2
- net CH340_USB_DN: track 0.00 -> 15.3 mm, vias 1 -> 2
- net CH340_USB_DP: track 0.13 -> 15.1 mm, vias 1 -> 2
- net GND: track 86.3 -> 94.9 mm, vias 36 -> 38
- net Net-(U2-RXD): track 0.00 -> 3.86 mm, vias 0 -> 1
- net Net-(U2-V3): track 0.00 -> 3.84 mm, vias 0 -> 1
- net Net-(J3-CC2): track 0.00 -> 3.40 mm, vias 0 -> 1
- net Net-(J3-CC1): track 0.00 -> 3.12 mm, vias 0 -> 1
- net Net-(U2-TXD): track 0.00 -> 3.07 mm, vias 0 -> 1

Commit message: update
Routing:
- net STLINK_3V3: track 0.00 -> 40.2 mm, vias 0 -> 3
- net REG_3V3: track 9.20 -> 35.7 mm, vias 2 -> 5
- net STM32_3V3: track 0.00 -> 26.1 mm, vias 0 -> 3
- net GND: track 94.9 -> 103.1 mm, vias 38 -> 40
- net NRST: track 0.00 -> 6.83 mm
