File: stm32pcb.kicad_pcb (KiCad board)
At the start: 2 copper layers, 61.1 x 40.7 mm, 45 parts, among them J1 USB_C_Receptacle_USB2.0_16P, J2 Conn_01x04_Pin, J3 USB_C_Receptacle_USB2.0_16P, J4 Conn_01x12_Pin, J5 Conn_01x12_Pin, J6 Conn_01x12_Pin, J7 Conn_01x12_Pin, SW1 SW_Push_DPDT, SW2 SW_Push_DPDT, SW3 SW_Push_DPDT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

Commit message: update
Routing:
- net STM32_3V3: track 26.1 -> 111.5 mm, vias 3 -> 10
- net SWDIO: track 0.00 -> 34.3 mm, vias 0 -> 2
- net SWCLK: track 0.00 -> 30.6 mm
- net GND: track 103.1 -> 109.0 mm, vias 40 -> 42
- net USB_DP: track 36.3 -> 42.2 mm
- net USB_DN: track 36.4 -> 40.6 mm
- net STLINK_3V3: track 40.2 -> 40.3 mm, vias 3 -> 5

Commit message: update
Parts:
- added R13: 22Ω, Resistor_SMD:R_1206_3216Metric, B.Cu at (172.2, 98.9)
- added R14: 22Ω, Resistor_SMD:R_1206_3216Metric, B.Cu at (172.2, 96.5)
- moved R4 11.4 mm to (187.1, 97.6)
- moved R3 10.5 mm to (198.1, 96.9)
Connections:
- J2 pad 3: SWDIO -> Net-(J2-Pin_3)
- J2 pad 4: SWCLK -> Net-(J2-Pin_4)
Routing:
- net CH340_TX: track 0.00 -> 32.8 mm, vias 0 -> 2
- net CH340_RX: track 0.00 -> 28.7 mm, vias 0 -> 1
- net STM32_3V3: track 111.5 -> 125.0 mm, vias 10 -> 13
- net Net-(R3-Pad2): track 0.00 -> 11.6 mm
- net Net-(R4-Pad2): track 0.00 -> 11.4 mm
- net SWDIO: track 34.3 -> 23.7 mm, vias 2 -> 1
- net SWCLK: track 30.6 -> 20.3 mm, vias 0 -> 1
- net Net-(J2-Pin_4): track 0.00 -> 7.38 mm, vias 0 -> 1
- net Net-(J2-Pin_3): track 0.00 -> 7.26 mm, vias 0 -> 1
- net GND: track 109.0 -> 114.9 mm, vias 42 -> 46

Commit message: update
Parts:
- moved C10 0.95 mm to (198.1, 84.2), turned to -90 degrees
Connections:
- J4 pad 3: unconnected-(J4-Pin_3-Pad3) -> OSC32_IN
Routing:
- net STM32_3V3: track 125.0 -> 284.4 mm, vias 13 -> 15
- net OSC32_IN: track 8.80 -> 49.4 mm, vias 0 -> 2
- net OSC32_OUT: track 8.88 -> 47.7 mm, vias 0 -> 2
- net OSC_IN: track 7.54 -> 44.5 mm, vias 0 -> 2
- net OSC_OUT: track 7.44 -> 42.8 mm, vias 0 -> 2
- net NRST: track 6.83 -> 41.6 mm, vias 0 -> 3
- net PB2_BOOT1: track 0.00 -> 31.9 mm, vias 0 -> 1
- net Net-(J4-Pin_2): track 0.00 -> 21.5 mm
- net Net-(J4-Pin_1): track 0.00 -> 21.1 mm
- net Net-(J4-Pin_12): track 0.00 -> 18.7 mm
- net Net-(J5-Pin_1): track 0.00 -> 18.5 mm
- net Net-(J4-Pin_11): track 0.00 -> 17.9 mm
- net Net-(J6-Pin_1): track 0.00 -> 17.7 mm
- net Net-(J5-Pin_2): track 0.00 -> 17.6 mm
- net Net-(J4-Pin_10): track 0.00 -> 17.0 mm
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- added copper zone on B.Cu, net GND
- added copper zone on F.Cu, net GND

Commit message: update
Routing:
- net GND: track 120.3 -> 121.1 mm, vias 69 -> 78
Changed lines of the file:
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@@
 	)
 	(segment
+		(start 203.665621 86.751777)
+		(end 204.019175 86.398223)
+		(width 0.3048)
+		(layer "F.Cu")
+		(net 3)
+	)
+	(segment
 		(start 191.7375 82.3875)
 		(end 192.09 82.74)
@@
 	)
 	(segment
+		(start 206.121751 93.421751)
+		(end 206.146751 93.421751)
+		(width 0.3048)
+		(layer "F.Cu")
+		(net 3)
+	)
+	(segment
 		(start 162.475 79.15)
 		(end 162.6 79.275)
@@
 	)
 	(segment
+		(start 205.812068 84.746751)
+		(end 205.812068 84.837068)
+		(width 0.3048)
+		(layer "F.Cu")
+		(net 3)
+	)
+	(segment
 		(start 207.35 87.525)
 		(end 207.625 87.8)
@@
 	)
 	(segment
+		(start 206.223223 86.398223)
+		(end 206.55 86.725)
+		(width 0.3048)
+		(layer "F.Cu")
+		(net 3)
+	)
+	(segment
 		(start 183.02 67.85)
 		(end 183.02 69.88)
@@
 	)
 	(segment
-		(start 206.121751 93.421751)
-		(end 204.678249 93.421751)
-		(width 0.2)
-		(layer "F.Cu")
-		(net 3)
-	)
-	(segment
-		(start 204.571751 93.528249)
-		(end 204.625 93.475)
-		(width 0.2)
+		(start 201.261459 86.751777)
+		(end 203.665621 86.751777)
+		(width 0.3048)
 		(layer "F.Cu")
 		(net 3)
 	)
 	(segment
-		(start 204.940317 85.6)
-		(end 204.817398 85.6)
-		(width 0.2)
+		(start 205.862068 87.878249)
+		(end 205.862068 88.337068)
+		(width 0.3048)
 		(layer "F.Cu")
 		(net 3)
@@
 	)
 	(segment
-		(start 202.792094 86.398223)
-		(end 202.640317 86.55)
-		(width 0.2)
-		(layer "F.Cu")
-		(net 3)
-	)
-	(segment
 		(start 207.625 84.25)
 		(end 207.625 84.9)
@@
 	)
 	(segment
-		(start 205.793566 84.746751)
-		(end 204.940317 85.6)
-		(width 0.2)
-		(layer "F.Cu")
-		(net 3)
-	)
-	(segment
-		(start 204.720952 87.1)
-		(end 204.019175 86.398223)
-		(width 0.2)
-		(layer "F.Cu")
-		(net 3)
-	)
-	(segment
 		(start 205.9 90.125)
 		(end 205.9 91.05)
@@
 	)
 	(segment
-		(start 204.915317 87.1)
-		(end 204.720952 87.1)
-		(width 0.2)
-		(layer "F.Cu")
-		(net 3)
-	)
-	(segment
 		(start 199.55 91.325)
 		(end 200.4 90.475)
@@
 	)
 	(segment
-		(start 205.693566 87.878249)
-		(end 204.915317 87.1)
-		(width 0.2)
-		(layer "F.Cu")
-		(net 3)
-	)
-	(segment
 		(start 161.05 82.525953)
 		(end 160.124047 81.6)
@@
 	)
 	(segment
+		(start 205.862068 88.337068)
+		(end 206.775 89.25)
+		(width 0.3048)
+		(layer "F.Cu")
+		(net 3)
+	)
+	(segment
 		(start 161.025 78.4548)
 		(end 161.025 76.75)
@@
 	)
 	(segment
-		(start 167.2 79.15)
-		(end 165.475 79.15)
+		(start 205.812068 84.837068)
+		(end 206.75 85.775)
 		(width 0.3048)
 		(layer "F.Cu")
@@
 	)
 	(segment
-		(start 201.261459 86.751777)
-		(end 202.43854 86.751777)
-		(width 0.2)
+		(start 206.146751 93.421751)
+		(end 207.1 94.375)
+		(width 0.3048)
+		(layer "F.Cu")
+		(net 3)
+	)
+	(segment
+		(start 167.2 79.15)
+		(end 165.475 79.15)
+		(width 0.3048)
 		(layer "F.Cu")
 		(net 3)
@@
 	)
 	(segment
-		(start 204.817398 85.6)
-		(end 204.019175 86.398223)
-		(width 0.2)
-		(layer "F.Cu")
-		(net 3)
-	)
-	(segment
 		(start 190.791927 87.903858)
 		(end 189.825 87.903858)
@@
 	(segment
 		(start 204.571751 94.971751)
-		(end 204.571751 93.528249)
-		(width 0.2)
-		(layer "F.Cu")
-		(net 3)
-	)
-	(segment
-		(start 166.445 67.83)
-		(end 165.625 68.65)
+		(end 204.646751 94.971751)
 		(width 0.3048)
 		(layer "F.Cu")
@@
 	)
 	(segment
-		(start 161.05 92.1048)
-		(end 160.3548 92.8)
+		(start 204.646751 94.971751)
+		(end 205.575 95.9)
 		(width 0.3048)
 		(layer "F.Cu")
@@
 	)
 	(segment
-		(start 204.678249 93.421751)
-		(end 204.625 93.475)
-		(width 0.2)
+		(start 166.445 67.83)
+		(end 165.625 68.65)
+		(width 0.3048)
 		(layer "F.Cu")
 		(net 3)
 	)
 	(segment
-		(start 204.019175 86.398223)
-		(end 202.792094 86.398223)
-		(width 0.2)
+		(start 161.05 92.1048)
+		(end 160.3548 92.8)
+		(width 0.3048)
 		(layer "F.Cu")
 		(net 3)
@@
 	)
 	(segment
+		(start 204.019175 86.398223)
+		(end 206.223223 86.398223)
+		(width 0.3048)
+		(layer "F.Cu")
+		(net 3)
+	)
+	(segment
 		(start 167.75 67.7)
 		(end 166.975 66.925)
@@
 		(net 3)
 	)
-	(segment
-		(start 202.43854 86.751777)
-		(end 202.640317 86.55)
-		(width 0.2)
-		(layer "F.Cu")
-		(net 3)
-	)
 	(via
 		(at 181.4 88.95)
@@
 	)
 	(via
+		(at 171.86 97.91)
+		(size 0.6)
+		(drill 0.3)
+		(layers "F.Cu" "B.Cu")
+		(net 3)
+	)
+	(via
 		(at 206.375 91.525)
 		(size 0.6)
@@
 	)
 	(via
-		(at 204.915317 87.1)
+		(at 203.775 81.725)
 		(size 0.6)
 		(drill 0.3)
@@
 	)
 	(via
-		(at 203.775 81.725)
+		(at 207.1 94.375)
 		(size 0.6)
 		(drill 0.3)
@@
 	)
 	(via
-		(at 207.1 94.375)
+		(at 191.904659 66.86436)
 		(size 0.6)
 		(drill 0.3)
 		(layers "F.Cu" "B.Cu")
-		(free yes)
 		(net 3)
 	)
@@
 	)
 	(via
+		(at 174.7 66.81)
+		(size 0.6)
+		(drill 0.3)
+		(layers "F.Cu" "B.Cu")
+		(net 3)
+	)
+	(via
 		(at 168.1 80.925)
 		(size 0.6)
@@
 	)
 	(via
-		(at 189.87 70.84)
+		(at 194.44 66.87)
 		(size 0.6)
 		(drill 0.3)
@@
 	)
 	(via
-		(at 204.025 96.675)
+		(at 189.87 70.84)
 		(size 0.6)
 		(drill 0.3)
 		(layers "F.Cu" "B.Cu")
-		(free yes)
 		(net 3)
 	)
 	(via
-		(at 204.625 93.475)
+		(at 204.025 96.675)
 		(size 0.6)
 		(drill 0.3)
@@
 	)
 	(via
+		(at 213.02 104.23)
+		(size 0.6)
+		(drill 0.3)
+		(layers "F.Cu" "B.Cu")
+		(net 3)
+	)
+	(via
 		(at 202.16 100.69)
 		(size 0.6)
@@
 	)
 	(via
+		(at 191.89 104.12)
+		(size 0.6)
+		(drill 0.3)
+		(layers "F.Cu" "B.Cu")
+		(net 3)
+	)
+	(via
 		(at 202.8 95.45)
 		(size 0.6)
@@
 	)
 	(via
-		(at 204.940317 85.6)
+		(at 167.92 95.05)
 		(size 0.6)
 		(drill 0.3)
 		(layers "F.Cu" "B.Cu")
-		(free yes)
 		(net 3)
 	)
@@
 	)
 	(via
+		(at 164.73 74.98)
+		(size 0.6)
+		(drill 0.3)
+		(layers "F.Cu" "B.Cu")
+		(net 3)
+	)
+	(via
 		(at 191.39 101.36)
 		(size 0.6)
@@
 	)
 	(via
+		(at 186.93 104.22)
+		(size 0.6)
+		(drill 0.3)
+		(layers "F.Cu" "B.Cu")
+		(net 3)
+	)
+	(via
 		(at 206.75 85.775)
 		(size 0.6)
@@
 	)
 	(via
+		(at 194.59 104.16)
+		(size 0.6)
+		(drill 0.3)
+		(layers "F.Cu" "B.Cu")
+		(net 3)
+	)
+	(via
 		(at 179.19 83.69)
 		(size 0.6)
@@
 	)
 	(via
-		(at 202.640317 86.55)
+		(at 201 93.65)
 		(size 0.6)
 		(drill 0.3)
@@
 	)
 	(via
-		(at 201 93.65)
+		(at 205.1 81.725)
 		(size 0.6)
 		(drill 0.3)
@@
 	)
 	(via
-		(at 205.1 81.725)
+		(at 191.34 96.44)
+		(size 0.6)
+		(drill 0.3)
+		(layers "F.Cu" "B.Cu")
+		(net 3)
+	)
+	(via
+		(at 213.66 66.35)
 		(size 0.6)
 		(drill 0.3)
 		(layers "F.Cu" "B.Cu")
-		(free yes)
 		(net 3)
 	)
@@
 	)
 	(via
+		(at 175.55 90.52)
+		(size 0.6)
+		(drill 0.3)
+		(layers "F.Cu" "B.Cu")
+		(net 3)
+	)
+	(via
 		(at 166.975 66.925)
 		(size 0.6)
@@
 		(hatch edge 0.5)
 		(connect_pads
-			(clearance 0.5)
+			(clearance 0.254)
 		)
 		(min_thickness 0.25)
@@
 			)
 		)
+	)
+	(zone
+		(net 0)
+		(net_name "")
+		(layers "F.Cu" "B.Cu")
+		(hatch edge 0.5)
+		(connect_pads
+			(clearance 0)
+		)
+		(min_thickness 0.25)
+		(filled_areas_thickness no)
+		(keepout
+			(tracks allowed)
+			(vias allowed)
+			(pads allowed)
+			(copperpour not_allowed)
+			(footprints allowed)
+		)
+		(placement
+			(enabled no)
+			(sheetname "/")
+		)
+		(fill
+			(thermal_gap 0.5)
+			(thermal_bridge_width 0.5)
+		)
+		(polygon
+			(pts
+				(xy 204.63 82.17) (xy 207.04 84.58) (xy 205.32 86.34) (xy 207.09 88.05) (xy 204.64 90.52) (xy 207.36 93.26)
+				(xy 204.43 96.21) (xy 200.14 91.85) (xy 201.01 90.98) (xy 201.01 89.36) (xy 199.03 87.67) (xy 197.33 87.67)
+				(xy 197.28 85.7) (xy 200.48 85.66)
+			)
+		)

Commit message: update
Routing:
- net USB_VBUS: track 15.1 -> 23.1 mm
- net STM32_3V3: track 284.4 -> 287.0 mm
- net Net-(D1-A): track 0.00 -> 2.35 mm, vias 0 -> 1
- net Net-(D2-A): track 0.00 -> 2.34 mm, vias 0 -> 1
- net USB_DP: track 42.2 -> 43.8 mm
- net GND: track 121.1 -> 122.5 mm, vias 78 -> 80
- net NRST: track 41.6 -> 42.9 mm
- net Net-(J3-CC2): track 3.40 -> 4.42 mm
Other:
- outline, holes or cut-outs redrawn
- board text added: "1"
- board text added: "10"
- board text added: "11"
- board text added: "12"
- board text added: "13"
- board text added: "14"
- board text added: "15"
- board text added: "16"
- board text added: "17"
- board text added: "18"
- board text added: "19"
- board text added: "2"
- board text added: "20"
- board text added: "21"
- board text added: "22"
- board text added: "23"
- board text added: "24"
- board text added: "25"
- board text added: "26"
- board text added: "27"
- board text added: "28"
- board text added: "29"
- board text added: "3"
- board text added: "30"
- board text added: "31"
- board text added: "32"
- board text added: "33"
- board text added: "34"
- board text added: "35"
- board text added: "36"
- board text added: "37"
- board text added: "38"
- board text added: "39"
- board text added: "3V3"
- board text added: "4"
- board text added: "40"
- board text added: "41"
- board text added: "42"
- board text added: "43"
- board text added: "44"
- board text added: "45"
- board text added: "46"
- board text added: "47"
- board text added: "48"
- board text added: "5"
- board text added: "6"
- board text added: "7"
- board text added: "8"
- board text added: "9"
- board text added: "GND"
- board text added: "Power Select"
- board text added: "REG"
- board text added: "REG-3V3"
- board text added: "STL"
- board text added: "STL-3v3"
- board text added: "STLink"
- board text added: "SWCLK"
- board text added: "SWDIO"

Commit message: update
Parts:
- SW3, SW4, SW5: moved to F.Cu
- moved SW5 1.52 mm to (183.7, 73.7)
- moved SW3 1.01 mm to (192.1, 96.9)
Routing:
- net STM32_3V3: track 287.0 -> 294.9 mm, vias 15 -> 13
- net GND: track 122.5 -> 115.9 mm, vias 80 -> 69
- net SWCLK: track 32.7 -> 35.1 mm
- net Net-(J7-Pin_2): track 16.9 -> 18.7 mm
- net Net-(J7-Pin_4): track 15.3 -> 16.9 mm
- net Net-(J7-Pin_3): track 16.6 -> 17.7 mm
- net NRST: track 42.9 -> 42.0 mm, vias 3 -> 4
- net Net-(J7-Pin_6): track 13.6 -> 14.4 mm
- net Net-(J7-Pin_7): track 14.0 -> 14.6 mm
- net Net-(J7-Pin_5): track 14.4 -> 15.0 mm
- net Net-(R4-Pad2): track 11.4 -> 11.2 mm, vias 0 -> 1
- net Net-(R3-Pad2): track 11.6 -> 11.8 mm, vias 0 -> 1

Commit message: update
Parts:
- moved R3 6.22 mm to (192.1, 95.0)
- moved R4 4.56 mm to (183.4, 95.1)
- moved SW4 1.30 mm to (183.4, 96.2)
- moved SW3 0.68 mm to (192.1, 96.2)
Routing:
- net Net-(R3-Pad2): track 11.8 -> 7.00 mm
- net GND: track 115.9 -> 120.5 mm, vias 69 -> 71
- net Net-(R4-Pad2): track 11.2 -> 7.67 mm
- net BOOT0: track 16.9 -> 20.2 mm
- net STM32_3V3: track 294.9 -> 296.9 mm
- net PB2_BOOT1: track 31.9 -> 33.7 mm
- net Net-(J7-Pin_2): track 18.7 -> 20.1 mm
- net Net-(J7-Pin_4): track 16.9 -> 15.7 mm
- net SWCLK: track 35.1 -> 36.1 mm, vias 1 -> 2
- net Net-(J7-Pin_7): track 14.6 -> 14.0 mm
- net Net-(J7-Pin_10): track 16.5 -> 17.1 mm
- net Net-(J7-Pin_5): track 15.0 -> 14.4 mm
Other:
- board text added: "Boot0"
- board text added: "Boot1"
- board text added: "Reset"

Commit message: update
Routing:
- net GND: vias 71 -> 75
Other:
- board text added: "CH340-USB"
- board text added: "Off"
- board text added: "On"
- board text added: "STL-3V3"
- board text added: "STM32-USB"
- board text removed: "STL-3v3"
