File: stm32pcb.kicad_sch (KiCad schematic)
At the start: 11 parts, among them J1 USB_C_Receptacle_USB2.0_16P, J2 Conn_01x04_Pin, J3 USB_C_Receptacle_USB2.0_16P, SW2 SW_Push_DPDT, U1 STM32F103C_8-B_Tx, U2 CH340C, U3 AMS1117-3.3

Commit message: 2
Parts:
- added C3: 100n, Capacitor_SMD:C_0805_2012Metric, symbol Device:C
- added SW1: SW_Push_DPDT, Button_Switch_SMD:SW_DPDT_CK_JS202011JCQN, symbol Switch:SW_Push_DPDT
- C1, C2: footprint (none) -> Capacitor_SMD:C_0805_2012Metric
Connections:
- net GND: now also J2.2 (Pin_2), C3.2
- net REG_3V3: now also SW1.3 (C), SW1.6 (C)
- net STLINK_3V3: now reaches J2.1 (Pin_1)
- net STLINK_3V3: now also C3.1, SW1.1 (A), SW1.4 (A)
- net SWDIO: now reaches J2.3 (Pin_3)
- net SWCLK: now reaches J2.4 (Pin_4)
- new net STM32_3V3: SW1.2 (B), SW1.5 (B)
Other:
- moved on the sheet: J2, U1

Commit message: update
Parts:
- added C4, C5: 22p, Capacitor_SMD:C_0805_2012Metric, symbol Device:C
- added C6, C7: 12pF, Capacitor_SMD:C_0805_2012Metric, symbol Device:C
- added Y1: 8MHz, symbol Device:Crystal_GND24
- added Y2: 32.768kHz, symbol Device:Crystal
- C1: value 10u -> 10uF
- C2: value 22u -> 22uF
- C3: value 100n -> 100nF
- R1, R2: value R -> 5.1kΩ
Connections:
- net GND: now also C4.2, C5.2, C6.2, C7.2, Y1.2 (G), Y1.4 (G)
- new net OSC32_IN: C6.1, Y2.1
- new net OSC32_OUT: C7.1, Y2.2
- new net OSC_IN: C4.1, Y1.1
- new net OSC_OUT: C5.1, Y1.3
Other:
- note added: "HSE"
- note added: "LSE"
- note added: "Power Selector"
- note added: "Regulator Power"
- note added: "ST-Link Interface"
- note added: "USB"
- moved on the sheet: C1, C2, C3, J1, J2, R1, R2, SW1, SW2, U1, U3

Commit message: update
Parts:
- SW1: footprint Button_Switch_SMD:SW_DPDT_CK_JS202011JCQN -> lcsc:SW-SMD_6P-L9.1-W3.5-P2.50
- Y1: footprint (none) -> Crystal:Crystal_SMD_3225-4Pin_3.2x2.5mm
- Y2: footprint (none) -> Crystal:Crystal_SMD_3215-2Pin_3.2x1.5mm
Other:
- moved on the sheet: C4, C5, C6, C7, Y1, Y2

Commit message: update
Parts:
- added C10, C11, C12, C8, C9: 100nF, Capacitor_SMD:C_0805_2012Metric, symbol Device:C
- added D1, D2: LED, symbol Device:LED
- added J4: Conn_01x12_Pin, symbol Connector:Conn_01x12_Pin
- added R3, R4, R7: 10kΩ, Resistor_SMD:R_1206_3216Metric, symbol Device:R
- added R5, R6: 1kΩ, Resistor_SMD:R_1206_3216Metric, symbol Device:R
- added R8: 1.5kΩ, Resistor_SMD:R_1206_3216Metric, symbol Device:R
- added SW3, SW4: SW_Push_DPDT, Button_Switch_SMD:SW_DPDT_CK_JS202011JCQN, symbol Switch:SW_Push_DPDT
- added SW5: TS-1088-AR02016, lcsc:SW-SMD_L3.9-W3.0-P4.45, symbol lcsc:TS-1088-AR02016
Connections:
- net GND: now also U1.23 (VSS), U1.35 (VSS), U1.47 (VSS), U1.8 (VSSA), C10.2, C11.2, C12.2, C8.2, C9.2, D1.1 (K), D2.1 (K), J4.8 (Pin_8), SW3.3 (C), SW3.6 (C), SW4.3 (C), SW4.6 (C), SW5.1
- net REG_3V3: now also R5.2
- net STLINK_3V3: now also R6.2
- net STM32_3V3: now also U1.24 (VDD), U1.36 (VDD), U1.48 (VDD), U1.9 (VDDA), C10.1, C11.1, C8.1, C9.1, J4.9 (Pin_9), R7.2, R8.2, SW3.1 (A), SW3.4 (A), SW4.1 (A), SW4.4 (A)
- net at U1.1 (VBAT): now also J4.1 (Pin_1)
- net at U1.10 (PA0): now also J4.10 (Pin_10)
- net at U1.11 (PA1): now also J4.11 (Pin_11)
- net at U1.12 (PA2): now also J4.12 (Pin_12)
- net at U1.2 (PC13): now also J4.2 (Pin_2)
- net PB2_BOOT1: now reaches U1.20 (PB2)
- net at U1.3 (PC14): now also J4.3 (Pin_3)
- net at U1.4 (PC15): now also J4.4 (Pin_4)
- net BOOT0: now reaches U1.44 (BOOT0)
- net BOOT0: now also R3.1, R4.1
- net at U1.5 (PD0): now also J4.5 (Pin_5)
- net at U1.6 (PD1): now also J4.6 (Pin_6)
- net NRST: now reaches U1.7 (NRST)
- net NRST: now also C12.1, J4.7 (Pin_7), R7.1, SW5.2
- net USB_DP: now reaches J1.A6 (D+)
- net USB_DP: now also J1.B6 (D+), R8.1
- net USB_DN: now reaches J1.A7 (D-)
- net USB_DN: now also J1.B7 (D-)
- new net: D1.2 (A), R5.1
- new net: R3.2, SW3.2 (B), SW3.5 (B)
- new net: R4.2, SW4.2 (B), SW4.5 (B)
- new net: D2.2 (A), R6.1
Other:
- note added: "BOOT"
- note added: "LED"
- note added: "RESET"
- note added: "SoC Power Filter"
- moved on the sheet: C1, C2, C4, C5, C6, C7, J3, SW1, SW2, U1, U2, U3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

Commit message: update
Parts:
- added C13, C14: 100nF, Capacitor_SMD:C_0805_2012Metric, symbol Device:C
- added J5, J6, J7: Conn_01x12_Pin, Connector_PinHeader_2.54mm:PinHeader_1x12_P2.54mm_Vertical, symbol Connector:Conn_01x12_Pin
- added R10, R9: 5.1kΩ, Resistor_SMD:R_1206_3216Metric, symbol Device:R
- added R11, R12: 220Ω, Resistor_SMD:R_1206_3216Metric, symbol Device:R
- D1, D2: footprint (none) -> LED_SMD:LED_0805_2012Metric
- J4: footprint (none) -> Connector_PinHeader_2.54mm:PinHeader_1x12_P2.54mm_Vertical
- SW2, SW3, SW4: footprint Button_Switch_SMD:SW_DPDT_CK_JS202011JCQN -> lcsc:SW-SMD_6P-L9.1-W3.5-P2.50
Connections:
- net BOOT0: now also J7.8 (Pin_8)
- net GND: now also J3.A1 (GND), J3.A12 (GND), J3.B1 (GND), J3.B12 (GND), J3.S1 (SHIELD), U2.1 (GND), C13.2, C14.2, J5.11 (Pin_11), J6.11 (Pin_11), J7.11 (Pin_11), R10.2, R9.2
- net OSC32_IN: now also U1.3 (PC14)
- net OSC32_OUT: now also J4.4 (Pin_4), U1.4 (PC15)
- net OSC_IN: now also J4.5 (Pin_5), U1.5 (PD0)
- net OSC_OUT: now also J4.6 (Pin_6), U1.6 (PD1)
- net PB2_BOOT1: now also J5.8 (Pin_8)
- net STM32_3V3: now also J5.12 (Pin_12), J6.12 (Pin_12), J7.12 (Pin_12)
- net SWCLK: now also U1.37 (PA14), J7.1 (Pin_1)
- net SWDIO: now also U1.34 (PA13), J6.10 (Pin_10)
- net USB_DN: now also U1.32 (PA11), J6.8 (Pin_8)
- net USB_DP: now also U1.33 (PA12), J6.9 (Pin_9)
- net CH340_USB_VBUS: now reaches J3.A4 (VBUS), J3.A9 (VBUS), J3.B4 (VBUS), J3.B9 (VBUS)
- net CH340_USB_VBUS: now also U2.16 (VCC), C14.1
- net at J3.A5 (CC1): now also R9.1
- net CH340_USB_DP: now reaches J3.A6 (D+)
- net CH340_USB_DP: now also J3.B6 (D+), U2.5 (UD+)
- net CH340_USB_DN: now reaches J3.A7 (D-)
- net CH340_USB_DN: now also J3.B7 (D-), U2.6 (UD-)
- net at J3.B5 (CC2): now also R10.1
- net at U1.13 (PA3): now also J5.1 (Pin_1)
- net at U1.14 (PA4): now also J5.2 (Pin_2)
- net at U1.15 (PA5): now also J5.3 (Pin_3)
- net at U1.16 (PA6): now also J5.4 (Pin_4)
- net at U1.17 (PA7): now also J5.5 (Pin_5)
- net at U1.18 (PB0): now also J5.6 (Pin_6)
- net at U1.19 (PB1): now also J5.7 (Pin_7)
- net at U1.21 (PB10): now also J5.9 (Pin_9)
- net at U1.22 (PB11): now also J5.10 (Pin_10)
- net at U1.25 (PB12): now also J6.1 (Pin_1)
- net at U1.26 (PB13): now also J6.2 (Pin_2)
- net at U1.27 (PB14): now also J6.3 (Pin_3)
- net at U1.28 (PB15): now also J6.4 (Pin_4)
- net at U1.29 (PA8): now also J6.5 (Pin_5)
- net at J4.3 (Pin_3): no longer U1.3 (PC14)
- net CH340_RX: now reaches U1.30 (PA9)
- net CH340_RX: now also J6.6 (Pin_6), R12.2
- net CH340_TX: now reaches U1.31 (PA10)
- net CH340_TX: now also J6.7 (Pin_7), R11.2
- net at U1.38 (PA15): now also J7.2 (Pin_2)
- net at U1.39 (PB3): now also J7.3 (Pin_3)
- net at U1.40 (PB4): now also J7.4 (Pin_4)
- net at U1.41 (PB5): now also J7.5 (Pin_5)
- net at U1.42 (PB6): now also J7.6 (Pin_6)
- net at U1.43 (PB7): now also J7.7 (Pin_7)
- net at U1.45 (PB8): now also J7.9 (Pin_9)
- net at U1.46 (PB9): now also J7.10 (Pin_10)
- net at U2.2 (TXD): now also R11.1
- net at U2.3 (RXD): now also R12.1
- net at U2.4 (V3): now also C13.1
Other:
- note added: "CH340"
- note added: "STM32"
- note added: "STM32 Power Filter"
- note removed: "SoC Power Filter"
- moved on the sheet: C12, J3, J4, R7, SW5, U1, U2

Commit message: update
Parts:
- J1, J3: footprint Connector_USB:USB_C_Receptacle_GCT_USB4105-xx-A_16P_TopMnt_Horizontal -> lcsc:USB-C-SMD_HH-16P-CB-TYPE-C
Connections:
- net BOOT0: no longer R4.1
- net PB2_BOOT1: now also R4.1
Changed lines of the file:
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@@
 		)
 	)
+	(global_label "PB2_BOOT1"
+		(shape input)
+		(at 111.76 194.31 180)
+		(fields_autoplaced yes)
+		(effects
+			(font
+				(size 1.27 1.27)
+			)
+			(justify right)
+		)
+		(property "Intersheetrefs" "${INTERSHEET_REFS}"
+			(at 97.9496 194.31 0)
+			(effects
+				(font
+					(size 1.27 1.27)
+				)
+				(justify right)
+				(hide yes)
+			)
+		)
+	)
 	(global_label "STM32_3V3"
 		(shape input)
@@
 		)
 	)
-	(global_label "BOOT0"
-		(shape input)
-		(at 111.76 194.31 180)
-		(fields_autoplaced yes)
-		(effects
-			(font
-				(size 1.27 1.27)
-			)
-			(justify right)
-		)
-		(property "Intersheetrefs" "${INTERSHEET_REFS}"
-			(at 102.6667 194.31 0)
-			(effects
-				(font
-					(size 1.27 1.27)
-				)
-				(justify right)
-				(hide yes)
-			)
-		)
-	)
 	(global_label "OSC_OUT"
 		(shape input)
@@
 			)
 		)
-		(property "Footprint" "Connector_USB:USB_C_Receptacle_GCT_USB4105-xx-A_16P_TopMnt_Horizontal"
+		(property "Footprint" "lcsc:USB-C-SMD_HH-16P-CB-TYPE-C"
 			(at 360.68 220.98 0)
 			(effects
@@
 			)
 		)
-		(property "Footprint" "Connector_USB:USB_C_Receptacle_GCT_USB4105-xx-A_16P_TopMnt_Horizontal"
+		(property "Footprint" "lcsc:USB-C-SMD_HH-16P-CB-TYPE-C"
 			(at 31.75 44.45 0)
 			(effects

Commit message: update
Parts:
- added R13, R14: 22Ω, Resistor_SMD:R_1206_3216Metric, symbol Device:R
Connections:
- net SWCLK: now also R14.2; no longer J2.4 (Pin_4)
- net SWDIO: now also R13.2; no longer J2.3 (Pin_3)
- new net: J2.3 (Pin_3), R13.1
- new net: J2.4 (Pin_4), R14.1
Changed lines of the file:
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@@
 	(wire
 		(pts
+			(xy 101.6 40.64) (xy 102.87 40.64)
+		)
+		(stroke
+			(width 0)
+			(type default)
+		)
+	)
+	(wire
+		(pts
 			(xy 116.84 257.81) (xy 123.19 257.81)
 		)
@@
 	(wire
 		(pts
+			(xy 101.6 38.1) (xy 102.87 38.1)
+		)
+		(stroke
+			(width 0)
+			(type default)
+		)
+	)
+	(wire
+		(pts
 			(xy 375.92 69.85) (xy 386.08 69.85)
 		)
@@
 		)
 	)
-	(global_label "SWCLK"
-		(shape input)
-		(at 93.98 40.64 0)
-		(fields_autoplaced yes)
-		(effects
-			(font
-				(size 1.27 1.27)
-			)
-			(justify left)
-		)
-		(property "Intersheetrefs" "${INTERSHEET_REFS}"
-			(at 103.1942 40.64 0)
-			(effects
-				(font
-					(size 1.27 1.27)
-				)
-				(justify left)
-				(hide yes)
-			)
-		)
-	)
 	(global_label "PB2_BOOT1"
 		(shape input)
@@
 		)
 	)
+	(global_label "SWCLK"
+		(shape input)
+		(at 102.87 40.64 0)
+		(fields_autoplaced yes)
+		(effects
+			(font
+				(size 1.27 1.27)
+			)
+			(justify left)
+		)
+		(property "Intersheetrefs" "${INTERSHEET_REFS}"
+			(at 112.0842 40.64 0)
+			(effects
+				(font
+					(size 1.27 1.27)
+				)
+				(justify left)
+				(hide yes)
+			)
+		)
+	)
 	(global_label "STM32_3V3"
 		(shape input)
@@
 		)
 	)
-	(global_label "SWDIO"
-		(shape input)
-		(at 93.98 38.1 0)
-		(fields_autoplaced yes)
-		(effects
-			(font
-				(size 1.27 1.27)
-			)
-			(justify left)
-		)
-		(property "Intersheetrefs" "${INTERSHEET_REFS}"
-			(at 102.8314 38.1 0)
-			(effects
-				(font
-					(size 1.27 1.27)
-				)
-				(justify left)
-				(hide yes)
-			)
-		)
-	)
 	(global_label "CH340_RX"
 		(shape input)
@@
 		)
 	)
+	(global_label "SWDIO"
+		(shape input)
+		(at 102.87 38.1 0)
+		(fields_autoplaced yes)
+		(effects
+			(font
+				(size 1.27 1.27)
+			)
+			(justify left)
+		)
+		(property "Intersheetrefs" "${INTERSHEET_REFS}"
+			(at 111.7214 38.1 0)
+			(effects
+				(font
+					(size 1.27 1.27)
+				)
+				(justify left)
+				(hide yes)
+			)
+		)
+	)
 	(global_label "CH340_RX"
 		(shape input)
@@
 	)
 	(symbol
+		(lib_id "Device:R")
+		(at 97.79 38.1 90)
+		(unit 1)
+		(exclude_from_sim no)
+		(in_bom yes)
+		(on_board yes)
+		(dnp no)
+		(property "Reference" "R13"
+			(at 88.646 36.83 90)
+			(effects
+				(font
+					(size 1.27 1.27)
+				)
+			)
+		)
+		(property "Value" "22Ω"
+			(at 92.964 36.83 90)
+			(effects
+				(font
+					(size 1.27 1.27)
+				)
+			)
+		)
+		(property "Footprint" "Resistor_SMD:R_1206_3216Metric"
+			(at 97.79 39.878 90)
+			(effects
+				(font
+					(size 1.27 1.27)
+				)
+				(hide yes)
+			)
+		)
+		(property "Datasheet" "~"
+			(at 97.79 38.1 0)
+			(effects
+				(font
+					(size 1.27 1.27)
+				)
+				(hide yes)
+			)
+		)
+		(property "Description" "Resistor"
+			(at 97.79 38.1 0)
+			(effects
+				(font
+					(size 1.27 1.27)
+				)
+				(hide yes)
+			)
+		)
+		(pin "1"
+		)
+		(pin "2"
+		)
+		(instances
+			(project "stm32pcb"
+				(path "/deb2f888-ee5e-42ae-a295-95cf39931a97"
+					(reference "R13")
+					(unit 1)
+				)
+			)
+		)
+	)
+	(symbol
 		(lib_id "Device:C")
 		(at 69.85 240.03 0)
@@
 					(unit 1)
 				)
+			)
+		)
+	)
+	(symbol
+		(lib_id "Device:R")
+		(at 97.79 40.64 90)
+		(unit 1)
+		(exclude_from_sim no)
+		(in_bom yes)
+		(on_board yes)
+		(dnp no)
+		(property "Reference" "R14"
+			(at 88.646 39.624 90)
+			(effects
+				(font
+					(size 1.27 1.27)
+				)
+			)
+		)
+		(property "Value" "22Ω"
+			(at 92.964 39.624 90)
+			(effects
+				(font
+					(size 1.27 1.27)
+				)
+			)
+		)
+		(property "Footprint" "Resistor_SMD:R_1206_3216Metric"
+			(at 97.79 42.418 90)
+			(effects
+				(font
+					(size 1.27 1.27)
+				)
+				(hide yes)
+			)
+		)
+		(property "Datasheet" "~"
+			(at 97.79 40.64 0)
+			(effects
+				(font
+					(size 1.27 1.27)
+				)
+				(hide yes)
+			)
+		)
+		(property "Description" "Resistor"
+			(at 97.79 40.64 0)
+			(effects
+				(font
+					(size 1.27 1.27)
+				)
+				(hide yes)
+			)
+		)
+		(pin "1"
+		)
+		(pin "2"
+		)
+		(instances
+			(project "stm32pcb"
+				(path "/deb2f888-ee5e-42ae-a295-95cf39931a97"
+					(reference "R14")
+					(unit 1)
+				)

Commit message: update
Connections:
- net OSC32_IN: now also J4.3 (Pin_3)
Changed lines of the file:
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@@
+	(wire
+		(pts
+			(xy 275.59 57.15) (xy 278.13 57.15)
+		)
+		(stroke
+			(width 0)
+			(type default)
+		)
+	)
 	(wire
 		(pts
